Commit message: Retraining with better gazebo model

File: pingpong-simulation/src/pingpang_gazebo/urdf/pingpang.urdf.xacro (robot description, xacro)
@@ -55,5 +55,4 @@
   </link>
   <joint name="move_joint" type="fixed">
-    <!-- <origin xyz="1.4 3.2 0.25" rpy="0 0 0" /> -->
     <origin xyz="1.4 3.4 0.005" rpy="0 0 0" />
     <parent link="world" />
@@ -67,9 +66,4 @@
       <material name="body"/>
     </visual>
-<!--     <collision>
-      <geometry>
-         <box size="0.02 0.02 0.6"/>
-      </geometry>
-    </collision> -->
     <inertial>
       <mass value="0.1" />
@@ -81,5 +75,4 @@
   <joint name="move_1_joint" type="prismatic">
     <origin xyz="0 0 0.245" rpy="0 0 0" />
-     <!-- <origin xyz="0 0 0.6" rpy="0 0 0" /> -->
     <axis xyz="1 0 0"/>
     <parent link="base_link_m" />
@@ -94,9 +87,4 @@
       <material name="body"/>
     </visual>
-<!--     <collision>
-      <geometry>
-         <box size="0.02 0.02 0.2"/>
-      </geometry>
-    </collision> -->
     <inertial>
       <mass value="0.1" />
@@ -120,9 +108,4 @@
       <material name="body"/>
     </visual>
-<!--     <collision>
-      <geometry>
-         <box size="0.2 0.01 0.2"/>
-      </geometry>
-    </collision> -->
     <inertial>
       <mass value="0.1" />
@@ -141,5 +124,4 @@
   <xacro:ur10_robot prefix="" joint_limited="false"/>
   <joint name="base_joint" type="fixed">
-    <!-- <origin xyz="-1 0.5 1" rpy="0 ${-degrees_90} 0 " /> -->
     <origin xyz="0.0 -0.165 0.0" rpy="3.1415926 ${degrees_90} 0 " />
     <parent link="move_2_link" />

File: pingpong-simulation/src/ur_description/urdf/ur10.urdf.xacro (robot description, xacro)
@@ -281,6 +281,25 @@
         </geometry>
           <origin rpy="0 0 ${pi/-2.0}" xyz="0.0 0.0 0.1"/>
-          <mass>1</mass>
+          <max_contacts>10000</max_contacts>
+          <surface>
+             <bounce>
+              <restitution_coefficient>1</restitution_coefficient>
+              <threshold>0.001</threshold>
+            </bounce>
+            <friction>
+              <ode>
+                <mu>0</mu>
+                <mu2>0</mu2>
+              </ode>
+            </friction>
+            <contact>
+              <ode>
+                <kp>10e8</kp>
+                <kd>100</kd>
+              </ode>
+            </contact>
+          </surface>
           <inertial>
+            <mass>1</mass>
            <inertia>
             <ixx>1</ixx>
@@ -297,10 +316,6 @@
       <material>Gazebo/Red</material>
       <selfCollide>true</selfCollide>
-      <kp>1000000.0</kp>
-      <kd>1.0</kd>
-      <mu1>1.2</mu1>
-      <mu2>1.2</mu2>
-      <maxVel>50000.0</maxVel>
-      <minDepth>0.001</minDepth>
+      <maxVel>5e10</maxVel>
+      <!-- <minDepth>0.001</minDepth> -->
     </gazebo>
 <!--         <gazebo reference="${prefix}ee_link">
